Commit message: various updates

File: Man4_RMURV2/RoVi_gazebo/src/rotors_simulator/rotors_description/urdf/hummingbird_base.xacro (robot description, xacro)
@@ -28,4 +28,25 @@
   <!-- Mount an ADIS16448 IMU. -->
   <xacro:default_imu namespace="${namespace}" parent_link="${namespace}/base_link" />
+  <!-- Mount a GPS -->
+  <!--xacro:default_gps namespace="${namespace}" parent_link="${namespace}/base_link" /-->
+  <xacro:default_pressure_sensor namespace="${namespace}" parent_link="${namespace}/base_link" />
+<!-- Mount a VI-sensor in front of the Hummingbird. -->
+  <xacro:camera_macro
+    namespace="${namespace}"
+    parent_link="${namespace}/base_link"
+    camera_suffix=""
+    frame_rate="30.0"
+    horizontal_fov="1.5"
+    image_width="800"
+    image_height="600"
+    image_format="R8G8B8"
+    min_distance="0.02"
+    max_distance="350"
+    noise_mean="0.0"
+    noise_stddev="0.007"
+    enable_visual="true">
+    <box size="0.02 0.02 0.02" />
+    <origin xyz="0 0 -0.055" rpy="0.0 90.0 0.0" />
+  </xacro:camera_macro>
   <xacro:if value="$(arg enable_ground_truth)">
     <xacro:ground_truth_imu_and_odometry namespace="${namespace}" parent_link="${namespace}/base_link" />

File: Man4_RMURV2/RoVi_gazebo/src/rotors_simulator/rotors_description/urdf/iris_base.xacro (robot description, xacro)
@@ -12,4 +12,6 @@
   <!-- Mount an ADIS16448 IMU. -->
   <xacro:default_imu namespace="${namespace}" parent_link="${namespace}/base_link" />
+  <!-- Mount a camera -->
+  <xacro:default_camera namespace="{namespace}" parent_link="${namespace}/base_link" />
   <xacro:if value="$(arg enable_ground_truth)">
     <xacro:ground_truth_imu_and_odometry namespace="${namespace}" parent_link="${namespace}/base_link" />

Commit message: Yaw works, also added new world

File: Man4_RMURV2/RoVi_gazebo/src/rotors_simulator/rotors_description/urdf/hummingbird_base.xacro (robot description, xacro)
@@ -47,5 +47,5 @@
     enable_visual="true">
     <box size="0.02 0.02 0.02" />
-    <origin xyz="0 0 -0.055" rpy="0.0 90.0 0.0" />
+    <origin xyz="0 0 -0.055" rpy="0.0 1.57079633 0.0" />
   </xacro:camera_macro>
   <xacro:if value="$(arg enable_ground_truth)">
